Commit message: Sensor upgrade, Write mapping.launch

File: src/my_robot/urdf/my_robot.xacro (robot description, xacro)
@@ -125,5 +125,5 @@
   </joint>
   <!-- link =  camera -->
-  <link name='camera'>
+  <link name='camera_link'>
     <pose>0 0 0 0 0 0</pose>
     <inertial>
@@ -151,8 +151,37 @@
   <!-- joint =  camera -->
   <joint type="fixed" name="camera_joint">
-    <origin xyz="0.2 0 0" rpy="0 0 0"/>
-    <child link="camera"/>
-    <parent link="chassis"/>
-    <axis xyz="0 1 0" rpy="0 0 0"/>
+    <origin xyz="0.1 0 0.1" rpy="0 0 0"/>
+    <child link="camera_link"/>
+    <parent link="chassis"/>
+    <axis xyz="0 1 0" rpy="0 0 0"/>
+  </joint>
+<!-- rgb-d camera -->
+<link name="camera_link_optical">
+     <visual>
+      <origin xyz="0 0 0" rpy="0 0 0"/>
+       <geometry>
+	<box size=".05 .05 .05"/>
+      </geometry>
+    </visual>
+    <inertial>
+      <mass value="0.1"/>
+      <origin xyz="0 0 0" rpy=" 0 0 0"/>
+      <inertia
+	  ixx="0.000001" ixy="0" ixz="0"
+	  iyy="0.000001" iyz="0"
+	  izz="0.000001"
+      />
+    </inertial>
+    <collision>
+      <origin xyz="0 0 0" rpy="0 0 0"/>
+       <geometry>
+	<box size=".05 .05 .05"/>
+      </geometry>
+    </collision>
+</link>
+  <joint name="camera_link_optical_joint" type="fixed">
+    <origin xyz="0.1 0 0.1" rpy="-1.5707 0  -1.5707" />
+    <parent link="camera_link"/>
+    <child link="camera_link_optical"/>
   </joint>
   <!-- link =  hokuyo -->

Commit message: Remove file from previous project , and add database file

File: src/my_robot/urdf/my_robot.xacro (robot description, xacro)
@@ -22,5 +22,5 @@
       <origin xyz="0 0 0" rpy=" 0 0 0"/>
       <geometry>
-        <box size=".4 .2 .1"/>
+        <box size=".4 .25 .1"/>
       </geometry>
     </collision>
@@ -28,5 +28,5 @@
       <origin xyz="0 0 0" rpy=" 0 0 0"/>
       <geometry>
-        <box size=".4 .2 .1"/>
+        <box size=".4 .25 .1"/>
       </geometry>
     </visual>
@@ -123,36 +123,4 @@
     <limit effort="10000" velocity="1000"/>
     <dynamics damping="1.0" friction="1.0"/>
-  </joint>
-  <!-- link =  camera -->
-  <link name='camera_link'>
-    <pose>0 0 0 0 0 0</pose>
-    <inertial>
-      <mass value="0.1"/>
-      <origin xyz="0.0 0 0" rpy=" 0 0 0"/>
-      <inertia
-          ixx="1e-6" ixy="0" ixz="0"
-          iyy="1e-6" iyz="0"
-          izz="1e-6"
-      />
-    </inertial>
-    <collision name='camera_collision'>
-      <origin xyz="0 0 0" rpy=" 0 0 0"/>
-      <geometry>
-        <box size = "0.05 0.05 0.05"/>
-      </geometry>
-    </collision>
-    <visual name='camera_visual'>
-      <origin xyz="0 0 0" rpy=" 0 0 0"/>
-      <geometry>
-        <box size = "0.05 0.05 0.05"/>
-      </geometry>
-    </visual>
-  </link>
-  <!-- joint =  camera -->
-  <joint type="fixed" name="camera_joint">
-    <origin xyz="0.1 0 0.1" rpy="0 0 0"/>
-    <child link="camera_link"/>
-    <parent link="chassis"/>
-    <axis xyz="0 1 0" rpy="0 0 0"/>
   </joint>
 <!-- rgb-d camera -->
@@ -181,7 +149,7 @@
 </link>
   <joint name="camera_link_optical_joint" type="fixed">
-    <origin xyz="0.1 0 0.1" rpy="-1.5707 0  -1.5707" />
-    <parent link="camera_link"/>
+    <origin xyz="0.075 0 0.075" rpy="-1.5707 0  -1.5707" />
     <child link="camera_link_optical"/>
+    <parent link="chassis"/>
   </joint>
   <!-- link =  hokuyo -->
@@ -212,5 +180,5 @@
   <!-- joint =  hokuyo_joint lidar  -->
   <joint type="fixed" name="hokuyo_joint">
-    <origin xyz="0.15 0.0 0.1" rpy="0 0 0"/>
+    <origin xyz="0.0 0.0 0.1" rpy="0 0 0"/>
     <child link="hokuyo"/>
     <parent link="chassis"/>
@@ -225,3 +193,9 @@
     <material>Gazebo/Green</material>
   </gazebo>
+  <gazebo reference="chassis">
+    <material>Gazebo/BlueTransparentOverlay</material>
+  </gazebo>
+  <gazebo reference="camera_link_optical">
+    <material>Gazebo/RedTransparent</material>
+  </gazebo>
 </robot>

Commit message: Rotate camera properly

File: src/my_robot/urdf/my_robot.xacro (robot description, xacro)
@@ -149,5 +149,5 @@
 </link>
   <joint name="camera_link_optical_joint" type="fixed">
-    <origin xyz="0.075 0 0.075" rpy="-1.5707 0  -1.5707" />
+    <origin xyz="0.075 0 0.075" rpy="0 0  0" />
     <child link="camera_link_optical"/>
     <parent link="chassis"/>
